Commit message: Update BionicHand.xacro

File: Code/Hand Urdf/BionicHand.xacro (robot description, xacro)
@@ -10,18 +10,47 @@
 <!-- Shape macros -->
 	<xacro:macro name="shape_box_lower_segment" params="">
-  	<geometry><box size="0.05 0.02 0.01"/></geometry>
+  	<geometry><box size="0.06 0.03 0.02"/></geometry>
 	</xacro:macro>
-<!-- Macro for a finger link -->
-<xacro:macro name="finger_link" params="name color_macro">
-  <link name="${name}">
-    <visual>
-      <xacro:shape_box_lower_segment/>
-			<!-- <box size="1 1 1"/> -->
-      <material name="${color_macro}"/>
-    </visual>
-  </link>
-</xacro:macro>
+  <!-- Redefine Shape top here -->
+  <xacro:macro name="shape_box_upper_segment" params="">
+  	<geometry><box size="0.06 0.03 0.02"/></geometry>
+	</xacro:macro>
+  <!-- Create Shape thumb lower here -->
+  <xacro:macro name="shape_box_thumb_lower_segment" params="">
+  	<geometry><box size="0.06 0.03 0.02"/></geometry>
+	</xacro:macro>
+<!-- Link Macros -->
+  <xacro:macro name="lower_link" params="name color_macro">
+    <link name="${name}">
+      <visual>
+        <origin xyz="0.025 0 0" rpy="0 0 0"/>
+        <xacro:shape_box_lower_segment/>
+        <material name="${color_macro}"/>
+      </visual>
+    </link>
+  </xacro:macro>
+  <xacro:macro name="upper_link" params="name color_macro">
+    <link name="${name}">
+      <visual>
+        <origin xyz="0.025 0 0" rpy="0 0 0"/>
+        <xacro:shape_box_upper_segment/>
+        <material name="${color_macro}"/>
+      </visual>
+    </link>
+  </xacro:macro>
+  <xacro:macro name="upper_link" params="name color_macro">
+    <link name="${name}">
+      <visual>
+        <origin xyz="0.025 0 0" rpy="0 0 0"/>
+        <xacro:shape_box_thumb_lower_segment/>
+        <material name="${color_macro}"/>
+      </visual>
+    </link>
+  </xacro:macro>
 <!-- Macro for a finger joint -->
-  <xacro:macro name="finger_joint" params="name parent child xyz rpy axis lower upper effort velocity">
+  <xacro:macro name="joint_limits" params="">
+    <limit lower="0" upper="1.57" effort="10" velocity="1"/>
+  </xacro:macro>
+  <xacro:macro name="finger_joint" params="name parent child xyz rpy axis">
     <joint name="${name}" type="revolute">
       <parent link="${parent}"/>
@@ -29,5 +58,5 @@
       <origin xyz="${xyz}" rpy="${rpy}"/>
       <axis xyz="${axis}"/>
-      <limit effort="${effort}" velocity="${velocity}" lower="${lower}" upper="${upper}"/>
+      <xacro:joint_limits/>
     </joint>
   </xacro:macro>
@@ -36,5 +65,5 @@
     <visual>
       <geometry>
-        <box size="0.1 0.1 0.02"/>
+        <box size="0.18 0.125 0.02"/>
       </geometry>
       <material>
@@ -44,13 +73,63 @@
   </link>
 <!-- Define fingers using macros -->
-	<xacro:finger_link name="index_lower" color_macro="color_white"/>
-	<xacro:finger_link name="finger_2_link" color_macro="color_yellow"/>
-	<xacro:finger_link name="finger_2_link" color_macro="color_yellow"/>
-	<xacro:finger_link name="finger_2_link" color_macro="color_yellow"/>
-  <xacro:finger_joint name="finger_1_joint" parent="base_link" child="finger_1_link"
-                      xyz="0 0 0.02" rpy="0 0 0" axis="0 1 0"
-                      lower="0" upper="1.57" effort="10" velocity="1"/>
-  <xacro:finger_joint name="finger_2_joint" parent="base_link" child="finger_2_link"
-                      xyz="0.05 0 0.02" rpy="0 0 0" axis="0 1 0"
-                      lower="0" upper="1.57" effort="10" velocity="1"/>
+  <!-- Mostly you will be messig with the xyz and positioning -->
+  <!-- xyz is where the joint rotates so make sure its at the end -->
+  <!-- look up or ask ai, idk figure out what axis and rpy does  -->
+	<xacro:lower_link name="index_lower" color_macro="color_white"/>
+	<xacro:upper_link name="index_upper" color_macro="color_yellow"/>
+  <xacro:finger_joint
+    name="index_base_lower_joint"
+    parent="base_link"
+    child="index_lower"
+    xyz="0.095 0.048 0" rpy="0 0 0" axis="0 1 0"
+  />
+  <xacro:finger_joint
+    name="index_upper_lower_joint"
+    parent="index_lower"
+    child="index_upper"
+    xyz="0.06 0 0" rpy="0 0 0" axis="0 1 0"
+  />
+  <!-- Copy the same format as above for each finger tweaking whatever is needed -->
+  <xacro:lower_link name="middle_lower" color_macro="color_white"/>
+	<xacro:upper_link name="middle_upper" color_macro="color_yellow"/>
+  <xacro:finger_joint
+    name="index_base_lower_joint"
+    parent="base_link"
+    child="middle_lower"
+    xyz="0.095 0.016 0" rpy="0 0 0" axis="0 1 0"
+  />
+  <xacro:finger_joint
+    name="index_upper_lower_joint"
+    parent="middle_lower"
+    child="middle_upper"
+    xyz="0.06 0 0" rpy="0 0 0" axis="0 1 0"
+  />
+  <xacro:lower_link name="ring_lower" color_macro="color_white"/>
+	<xacro:upper_link name="ring_upper" color_macro="color_yellow"/>
+  <xacro:finger_joint
+    name="index_base_lower_joint"
+    parent="base_link"
+    child="ring_lower"
+    xyz="0.095 -0.016 0" rpy="0 0 0" axis="0 1 0"
+  />
+  <xacro:finger_joint
+    name="index_upper_lower_joint"
+    parent="ring_lower"
+    child="ring_upper"
+    xyz="0.06 0 0" rpy="0 0 0" axis="0 1 0"
+  />
+  <xacro:lower_link name="pinky_lower" color_macro="color_white"/>
+	<xacro:upper_link name="pinky_upper" color_macro="color_yellow"/>
+  <xacro:finger_joint
+    name="index_base_lower_joint"
+    parent="base_link"
+    child="pinky_lower"
+    xyz="0.095 -0.048 0" rpy="0 0 0" axis="0 1 0"
+  />
+  <xacro:finger_joint
+    name="index_upper_lower_joint"
+    parent="pinky_lower"
+    child="pinky_upper"
+    xyz="0.06 0 0" rpy="0 0 0" axis="0 1 0"
+  />
 </robot>

Commit message: added some parsing

File: Code/Hand Urdf/BionicHand.xacro (robot description, xacro)
@@ -18,5 +18,5 @@
   <!-- Create Shape thumb lower here -->
   <xacro:macro name="shape_box_thumb_lower_segment" params="">
-  	<geometry><box size="0.06 0.03 0.02"/></geometry>
+  	<geometry><box size="0.08 0.03 0.02"/></geometry>
 	</xacro:macro>
 <!-- Link Macros -->
@@ -39,5 +39,5 @@
     </link>
   </xacro:macro>
-  <xacro:macro name="upper_link" params="name color_macro">
+  <xacro:macro name="thumb_link" params="name color_macro">
     <link name="${name}">
       <visual>
@@ -73,63 +73,70 @@
   </link>
 <!-- Define fingers using macros -->
-  <!-- Mostly you will be messig with the xyz and positioning -->
-  <!-- xyz is where the joint rotates so make sure its at the end -->
-  <!-- look up or ask ai, idk figure out what axis and rpy does  -->
-	<xacro:lower_link name="index_lower" color_macro="color_white"/>
-	<xacro:upper_link name="index_upper" color_macro="color_yellow"/>
-  <xacro:finger_joint
-    name="index_base_lower_joint"
+  <!-- Index -->
+	  <xacro:lower_link name="index_lower" color_macro="color_white"/>
+	  <xacro:upper_link name="index_upper" color_macro="color_yellow"/>
+    <xacro:finger_joint
+    name="index_lower_joint"
     parent="base_link"
     child="index_lower"
-    xyz="0.095 0.048 0" rpy="0 0 0" axis="0 1 0"
-  />
-  <xacro:finger_joint
-    name="index_upper_lower_joint"
-    parent="index_lower"
-    child="index_upper"
-    xyz="0.06 0 0" rpy="0 0 0" axis="0 1 0"
-  />
-  <!-- Copy the same format as above for each finger tweaking whatever is needed -->
-  <xacro:lower_link name="middle_lower" color_macro="color_white"/>
-	<xacro:upper_link name="middle_upper" color_macro="color_yellow"/>
-  <xacro:finger_joint
-    name="index_base_lower_joint"
+    xyz="0.095 0.048 0" rpy="0 0 0" axis="0 1 0"/>
+    <xacro:finger_joint
+      name="index_upper_joint"
+      parent="index_lower"
+      child="index_upper"
+      xyz="0.06 0 0" rpy="0 0 0" axis="0 1 0"/>
+  <!-- Middle -->
+    <xacro:lower_link name="middle_lower" color_macro="color_white"/>
+	  <xacro:upper_link name="middle_upper" color_macro="color_yellow"/>
+    <xacro:finger_joint
+    name="middle_lower_joint"
     parent="base_link"
     child="middle_lower"
-    xyz="0.095 0.016 0" rpy="0 0 0" axis="0 1 0"
-  />
-  <xacro:finger_joint
-    name="index_upper_lower_joint"
-    parent="middle_lower"
-    child="middle_upper"
-    xyz="0.06 0 0" rpy="0 0 0" axis="0 1 0"
-  />
-  <xacro:lower_link name="ring_lower" color_macro="color_white"/>
-	<xacro:upper_link name="ring_upper" color_macro="color_yellow"/>
-  <xacro:finger_joint
-    name="index_base_lower_joint"
+    xyz="0.095 0.016 0" rpy="0 0 0" axis="0 1 0"/>
+    <xacro:finger_joint
+      name="middle_upper_joint"
+      parent="middle_lower"
+      child="middle_upper"
+      xyz="0.06 0 0" rpy="0 0 0" axis="0 1 0"/>
+  <!-- Ring  -->
+    <xacro:lower_link name="ring_lower" color_macro="color_white"/>
+	  <xacro:upper_link name="ring_upper" color_macro="color_yellow"/>
+    <xacro:finger_joint
+    name="ring_lower_joint"
     parent="base_link"
     child="ring_lower"
-    xyz="0.095 -0.016 0" rpy="0 0 0" axis="0 1 0"
-  />
-  <xacro:finger_joint
-    name="index_upper_lower_joint"
-    parent="ring_lower"
-    child="ring_upper"
-    xyz="0.06 0 0" rpy="0 0 0" axis="0 1 0"
-  />
-  <xacro:lower_link name="pinky_lower" color_macro="color_white"/>
-	<xacro:upper_link name="pinky_upper" color_macro="color_yellow"/>
-  <xacro:finger_joint
-    name="index_base_lower_joint"
-    parent="base_link"
-    child="pinky_lower"
-    xyz="0.095 -0.048 0" rpy="0 0 0" axis="0 1 0"
-  />
-  <xacro:finger_joint
-    name="index_upper_lower_joint"
-    parent="pinky_lower"
-    child="pinky_upper"
-    xyz="0.06 0 0" rpy="0 0 0" axis="0 1 0"
-  />
+    xyz="0.095 -0.016 0" rpy="0 0 0" axis="0 1 0"/>
+    <xacro:finger_joint
+      name="ring_upper_joint"
+      parent="ring_lower"
+      child="ring_upper"
+      xyz="0.06 0 0" rpy="0 0 0" axis="0 1 0"/>
+  <!-- Pinky -->
+    <xacro:lower_link name="pinky_lower" color_macro="color_white"/>
+	  <xacro:upper_link name="pinky_upper" color_macro="color_yellow"/>
+    <xacro:finger_joint
+      name="pinky_lower_joint"
+      parent="base_link"
+      child="pinky_lower"
+      xyz="0.095 -0.048 0" rpy="0 0 0" axis="0 1 0"/>
+    <xacro:finger_joint
+      name="pinky_upper_joint"
+      parent="pinky_lower"
+      child="pinky_upper"
+      xyz="0.06 0 0" rpy="0 0 0" axis="0 1 0"/>
+  <!-- Thumb -->
+    <xacro:lower_link name="thumb_lower" color_macro="color_white"/>
+	  <xacro:upper_link name="thumb_upper" color_macro="color_yellow"/>
+    <xacro:finger_joint
+      name="thumb_lower_joint"
+      parent="base_link"
+      child="thumb_lower"
+      xyz="-0.02 0.055 0"
+      rpy="-0.78 0 1.57"
+      axis="0 1 0"/>
+    <xacro:finger_joint
+      name="thumb_upper_joint"
+      parent="thumb_lower"
+      child="thumb_upper"
+      xyz="0.06 0 0" rpy="0 0 0" axis="0 1 0"/>
 </robot>

Commit message: Recent

File: Code/Hand Urdf/BionicHand.xacro (robot description, xacro)
@@ -50,5 +50,5 @@
 <!-- Macro for a finger joint -->
   <xacro:macro name="joint_limits" params="">
-    <limit lower="0" upper="1.57" effort="10" velocity="1"/>
+    <limit lower="-1.57" upper="1.57" effort="10" velocity="1"/>
   </xacro:macro>
   <xacro:macro name="finger_joint" params="name parent child xyz rpy axis">
