Commit message: made it run off docker

File: hand-tracker/Code/Hand Urdf/BionicHand.xacro (robot description, xacro)
@@ -67,5 +67,5 @@
         <box size="0.18 0.125 0.02"/>
       </geometry>
-      <material>
+      <material name="color_orange">
         <color rgba="1 0.5 0 1"/>
       </material>
